Commit message: Joints homework

File: body2.urdf (robot description, URDF)
Before this commit: robot robot, 2 links, 1 joints
Links:
- added link BackLeg, mass 1; collision box size=1 1 1; visual box size=1 1 1
Joints:
- added joint Torso_BackLeg: type revolute, parent Torso, child BackLeg, origin xyz=1.0 0 1.0 rpy=0 0 0, axis 0 1 0, limit lower=-3.14159 upper=3.14159 effort=0.0 velocity=0.0
- joint Torso_FrontLeg: origin xyz=0 1 0 rpy=0 0 0 -> xyz=2.0 0 1.0 rpy=0 0 0

Commit message: Quad finished

File: body2.urdf (robot description, URDF)
Before this commit: robot robot, 3 links, 2 joints
Links:
- added link BackLowerLeg, mass 1; collision box size=0.2 0.2 1; visual box size=0.2 0.2 1
- added link FrontLowerLeg, mass 1; collision box size=0.2 0.2 1; visual box size=0.2 0.2 1
- added link LeftLeg, mass 1; collision box size=1 0.2 0.2; visual box size=1 0.2 0.2
- added link LeftLowerLeg, mass 1; collision box size=0.2 0.2 1; visual box size=0.2 0.2 1
- added link RightLeg, mass 1; collision box size=1 0.2 0.2; visual box size=1 0.2 0.2
- added link RightLowerLeg, mass 1; collision box size=0.2 0.2 1; visual box size=0.2 0.2 1
- link BackLeg: geometry collision box size=0.2 1 0.2; visual box size=0.2 1 0.2
- link FrontLeg: geometry collision box size=0.2 1 0.2; visual box size=0.2 1 0.2
Joints:
- added joint BackLeg_BackLowerLeg: type revolute, parent BackLeg, child BackLowerLeg, origin xyz=0 -1 0 rpy=0 0 0, axis 1 0 0, limit lower=-3.14159 upper=3.14159 effort=0.0 velocity=0.0
- added joint FrontLeg_FrontLowerLeg: type revolute, parent FrontLeg, child FrontLowerLeg, origin xyz=0 1 0 rpy=0 0 0, axis 1 0 0, limit lower=-3.14159 upper=3.14159 effort=0.0 velocity=0.0
- added joint LeftLeg_LeftLowerLeg: type revolute, parent LeftLeg, child LeftLowerLeg, origin xyz=-1 0 0 rpy=0 0 0, axis 0 1 0, limit lower=-3.14159 upper=3.14159 effort=0.0 velocity=0.0
- added joint RightLeg_RightLowerLeg: type revolute, parent RightLeg, child RightLowerLeg, origin xyz=1 0 0 rpy=0 0 0, axis 0 1 0, limit lower=-3.14159 upper=3.14159 effort=0.0 velocity=0.0
- added joint Torso_LeftLeg: type revolute, parent Torso, child LeftLeg, origin xyz=-0.5 0 1.0 rpy=0 0 0, axis 1 0 0, limit lower=-3.14159 upper=3.14159 effort=0.0 velocity=0.0
- added joint Torso_RightLeg: type revolute, parent Torso, child RightLeg, origin xyz=0.5 0 1.0 rpy=0 0 0, axis 1 0 0, limit lower=-3.14159 upper=3.14159 effort=0.0 velocity=0.0
- joint Torso_BackLeg: axis 0 1 0 -> 1 0 0; origin xyz=1.0 0 1.0 rpy=0 0 0 -> xyz=0 -0.5 1.0 rpy=0 0 0
- joint Torso_FrontLeg: axis 0 1 0 -> 1 0 0; origin xyz=2.0 0 1.0 rpy=0 0 0 -> xyz=0 0.5 1.0 rpy=0 0 0

Commit message: Hexapod started

File: body2.urdf (robot description, URDF)
Before this commit: robot robot, 9 links, 8 joints
Links:
- added link Mid1Leg, mass 1; collision box size=1 0.2 0.2; visual box size=1 0.2 0.2
- added link Mid1LowerLeg, mass 1; collision box size=0.2 0.2 1; visual box size=0.2 0.2 1
- added link Mid2Leg, mass 1; collision box size=1 0.2 0.2; visual box size=1 0.2 0.2
- added link Mid2LowerLeg, mass 1; collision box size=0.2 0.2 1; visual box size=0.2 0.2 1
- link Torso: geometry collision box size=1 2 1; visual box size=1 2 1
Joints:
- added joint Mid1Leg_Mid1LowerLeg: type revolute, parent Mid1Leg, child Mid1LowerLeg, origin xyz=-1 0 0 rpy=0 0 0, axis 0 1 0, limit lower=-3.14159 upper=3.14159 effort=0.0 velocity=0.0
- added joint Mid2Leg_Mid2LowerLeg: type revolute, parent Mid2Leg, child Mid2LowerLeg, origin xyz=1 0 0 rpy=0 0 0, axis 0 1 0, limit lower=-3.14159 upper=3.14159 effort=0.0 velocity=0.0
- added joint Torso_Mid1Leg: type revolute, parent Torso, child Mid1Leg, origin xyz=-0.5 0 1.0 rpy=0 0 0, axis 1 0 0, limit lower=-3.14159 upper=3.14159 effort=0.0 velocity=0.0
- added joint Torso_Mid2Leg: type revolute, parent Torso, child Mid2Leg, origin xyz=0.5 0 1.0 rpy=0 0 0, axis 1 0 0, limit lower=-3.14159 upper=3.14159 effort=0.0 velocity=0.0

Commit message: octopod

File: body2.urdf (robot description, URDF)
Before this commit: robot robot, 13 links, 12 joints
Links:
- added link Mid3Leg, mass 1; collision box size=1 0.2 0.2; visual box size=1 0.2 0.2
- added link Mid3LowerLeg, mass 1; collision box size=0.2 0.2 1; visual box size=0.2 0.2 1
- added link Mid4Leg, mass 1; collision box size=1 0.2 0.2; visual box size=1 0.2 0.2
- added link Mid4LowerLeg, mass 1; collision box size=0.2 0.2 1; visual box size=0.2 0.2 1
- link Torso: geometry collision box size=1 4 1; visual box size=1 4 1
Joints:
- added joint Mid3Leg_Mid3LowerLeg: type revolute, parent Mid3Leg, child Mid3LowerLeg, origin xyz=-1 0 0 rpy=0 0 0, axis 0 1 0, limit lower=-3.14159 upper=3.14159 effort=0.0 velocity=0.0
- added joint Mid4Leg_Mid4LowerLeg: type revolute, parent Mid4Leg, child Mid4LowerLeg, origin xyz=1 0 0 rpy=0 0 0, axis 0 1 0, limit lower=-3.14159 upper=3.14159 effort=0.0 velocity=0.0
- added joint Torso_Mid3Leg: type revolute, parent Torso, child Mid3Leg, origin xyz=-0.5 1 1 rpy=0 0 0, axis 0 1 0, limit lower=-3.14159 upper=3.14159 effort=0.0 velocity=0.0
- added joint Torso_Mid4Leg: type revolute, parent Torso, child Mid4Leg, origin xyz=0.5 1 1 rpy=0 0 0, axis 0 1 0, limit lower=-3.14159 upper=3.14159 effort=0.0 velocity=0.0
- joint Torso_BackLeg: origin xyz=0 -0.5 1.0 rpy=0 0 0 -> xyz=0 -2 1 rpy=0 0 0
- joint Torso_FrontLeg: origin xyz=0 0.5 1.0 rpy=0 0 0 -> xyz=0 2 1 rpy=0 0 0
- joint Torso_LeftLeg: axis 1 0 0 -> 0 1 0; origin xyz=-0.5 0 1.0 rpy=0 0 0 -> xyz=-0.5 -1 1 rpy=0 0 0
- joint Torso_Mid1Leg: axis 1 0 0 -> 0 1 0; origin xyz=-0.5 0 1.0 rpy=0 0 0 -> xyz=-0.5 0 1 rpy=0 0 0
- joint Torso_Mid2Leg: axis 1 0 0 -> 0 1 0; origin xyz=0.5 0 1.0 rpy=0 0 0 -> xyz=0.5 0 1 rpy=0 0 0
- joint Torso_RightLeg: axis 1 0 0 -> 0 1 0; origin xyz=0.5 0 1.0 rpy=0 0 0 -> xyz=0.5 -1 1 rpy=0 0 0

Commit message: 100 gens now

File: body2.urdf (robot description, URDF)
Before this commit: robot robot, 13 links, 12 joints
Joints:
- joint Torso_BackLeg: origin xyz=0 -0.5 1.0 rpy=0 0 0 -> xyz=0 -1 1 rpy=0 0 0
- joint Torso_FrontLeg: origin xyz=0 0.5 1.0 rpy=0 0 0 -> xyz=0 1 1 rpy=0 0 0
- joint Torso_LeftLeg: axis 1 0 0 -> 0 1 0; origin xyz=-0.5 0 1.0 rpy=0 0 0 -> xyz=-0.5 -0.5 1 rpy=0 0 0
- joint Torso_Mid1Leg: axis 1 0 0 -> 0 1 0; origin xyz=-0.5 0 1.0 rpy=0 0 0 -> xyz=-0.5 0.5 1 rpy=0 0 0
- joint Torso_Mid2Leg: axis 1 0 0 -> 0 1 0; origin xyz=0.5 0 1.0 rpy=0 0 0 -> xyz=0.5 0.5 1 rpy=0 0 0
- joint Torso_RightLeg: axis 1 0 0 -> 0 1 0; origin xyz=0.5 0 1.0 rpy=0 0 0 -> xyz=0.5 -0.5 1 rpy=0 0 0
